File: MosfetDriverOn2104/_saved_MosfetDriverOn210404.sch (KiCad schematic (older format))
At the start: 39 parts, among them J1 Screw_Terminal_01x02, Q1 IRF540N, Q2 IRF540N, U1 IR2104

Commit message: symbol changed!
Parts:
- removed U?: ATmega328P-AU, Package_QFP:TQFP-32_7x7mm_P0.8mm, symbol MosfetDriverOn210404-rescue:ATmega328P-AU-MCU_Microchip_ATmega
- added U?: ATmega328P-AU, Package_QFP:TQFP-32_7x7mm_P0.8mm, symbol MCU_Microchip_ATmega:ATmega328P-AU
Changed lines of the file:
@@
 Connection ~ 8350 2550
-$Comp
-L MosfetDriverOn210404-rescue:ATmega328P-AU-MCU_Microchip_ATmega U?
-U 1 1 5BCEBDA5
-P 2600 2700
-F 0 "U?" H 2150 4150 50  0000 C CNN
-F 1 "ATmega328P-AU" H 2500 1600 50  0000 C CNN
-F 2 "Package_QFP:TQFP-32_7x7mm_P0.8mm" H 2600 2700 50  0001 C CIN
-F 3 "http://ww1.microchip.com/downloads/en/DeviceDoc/ATmega328_P%20AVR%20MCU%20with%20picoPower%20Technology%20Data%20Sheet%2040001984A.pdf" H 2600 2700 50  0001 C CNN
-	1    2600 2700
-	1    0    0    -1
-$EndComp
 $Comp
 L Regulator_Switching:LM2576HVS-ADJ U?
@@
 	1    0    0    -1
 $EndComp
+$Comp
+L MCU_Microchip_ATmega:ATmega328P-AU U?
+U 1 1 5BCBA2FB
+P 3950 2450
+F 0 "U?" H 3950 864 50  0000 C CNN
+F 1 "ATmega328P-AU" H 3950 773 50  0000 C CNN
+F 2 "Package_QFP:TQFP-32_7x7mm_P0.8mm" H 3950 2450 50  0001 C CIN
+F 3 "http://ww1.microchip.com/downloads/en/DeviceDoc/ATmega328_P%20AVR%20MCU%20with%20picoPower%20Technology%20Data%20Sheet%2040001984A.pdf" H 3950 2450 50  0001 C CNN
+	1    3950 2450
+	1    0    0    -1
+$EndComp
