File: MosfetDriverOn2104/_saved_POwer & Connectors.sch (KiCad schematic (older format))
At the start: 25 parts, among them J1 I2C HDR, J10 ENCODER HDR, J2 AVR-ISP-6, J3 I2C HDR, J4 Screw_Terminal_01x02, J5 I2C HDR, J6 UART HDR, J7 5V HDR, J8 GND HDR, J9 servo hdr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

Commit message: Sorted PCB
Parts:
- J2: footprint Connector_PinHeader_2.54mm:PinHeader_1x04_P2.54mm_Vertical -> Connector_PinHeader_2.54mm:PinHeader_2x03_P2.54mm_Vertical
Changed lines of the file:
@@
 F 0 "J2" H 2000 4050 50  0000 R CNN
 F 1 "AVR-ISP-6" H 2350 3950 50  0000 R CNN
-F 2 "Connector_PinHeader_2.54mm:PinHeader_1x04_P2.54mm_Vertical" V 1650 3550 50  0001 C CNN
+F 2 "Connector_PinHeader_2.54mm:PinHeader_2x03_P2.54mm_Vertical" V 1650 3550 50  0001 C CNN
 F 3 " ~" H 625 2950 50  0001 C CNN
 	1    1900 3500
