File: MosfetDriverOn2104/controller.sch (KiCad schematic (older format))
At the start: 22 parts

Commit message: started routing
Parts:
- gave numbers to parts that had none: 22
Changed lines of the file:
@@
 $EndDescr
 $Comp
-L power:+5V #PWR?
+L power:+5V #PWR0101
 U 1 1 5BD0346C
 P 4350 3100
-F 0 "#PWR?" H 4350 2950 50  0001 C CNN
+F 0 "#PWR0101" H 4350 2950 50  0001 C CNN
 F 1 "+5V" H 4365 3273 50  0000 C CNN
 F 2 "" H 4350 3100 50  0001 C CNN
@@
 $EndComp
 $Comp
-L power:GND #PWR?
+L power:GND #PWR0102
 U 1 1 5BD03472
 P 4400 4900
-F 0 "#PWR?" H 4400 4650 50  0001 C CNN
+F 0 "#PWR0102" H 4400 4650 50  0001 C CNN
 F 1 "GND" H 4405 4727 50  0000 C CNN
 F 2 "" H 4400 4900 50  0001 C CNN
@@
 $EndComp
 $Comp
-L power:+5V #PWR?
+L power:+5V #PWR0103
 U 1 1 5BD03478
 P 3850 2500
-F 0 "#PWR?" H 3850 2350 50  0001 C CNN
+F 0 "#PWR0103" H 3850 2350 50  0001 C CNN
 F 1 "+5V" H 3865 2673 50  0000 C CNN
 F 2 "" H 3850 2500 50  0001 C CNN
@@
 $EndComp
 $Comp
-L power:GND #PWR?
+L power:GND #PWR0104
 U 1 1 5BD0347E
 P 3850 2900
-F 0 "#PWR?" H 3850 2650 50  0001 C CNN
+F 0 "#PWR0104" H 3850 2650 50  0001 C CNN
 F 1 "GND" H 3855 2727 50  0000 C CNN
 F 2 "" H 3850 2900 50  0001 C CNN
@@
 $EndComp
 $Comp
-L MosfetDriverOn210404-rescue:ATmega328P-AU-MCU_Microchip_ATmega U?
+L MosfetDriverOn210404-rescue:ATmega328P-AU-MCU_Microchip_ATmega U1
 U 1 1 5BD03484
 P 5400 3600
-F 0 "U?" H 4650 4450 50  0000 C CNN
+F 0 "U1" H 4650 4450 50  0000 C CNN
 F 1 "ATmega328P-AU-MCU_Microchip_ATmega" H 5350 2100 50  0000 C CNN
 F 2 "Package_QFP:TQFP-32_7x7mm_P0.8mm" H 5400 3300 50  0001 C CIN
@@
 $EndComp
 $Comp
-L Device:C_Small C?
+L Device:C_Small C1
 U 1 1 5BD0348B
 P 3700 2700
-F 0 "C?" H 3550 2750 50  0000 L CNN
+F 0 "C1" H 3550 2750 50  0000 L CNN
 F 1 "C_Small" H 3450 2650 50  0000 L CNN
 F 2 "Capacitor_SMD:C_0805_2012Metric" H 3700 2700 50  0001 C CNN
@@
 $EndComp
 $Comp
-L Device:C_Small C?
+L Device:C_Small C2
 U 1 1 5BD03492
 P 3850 2700
-F 0 "C?" H 3750 2750 50  0000 L CNN
+F 0 "C2" H 3750 2750 50  0000 L CNN
 F 1 "C_Small" H 3750 2650 50  0000 L CNN
 F 2 "Capacitor_SMD:C_0805_2012Metric" H 3850 2700 50  0001 C CNN
@@
 $EndComp
 $Comp
-L Device:CP_Small C?
+L Device:CP_Small C3
 U 1 1 5BD03499
 P 4000 2700
-F 0 "C?" H 4050 2750 50  0000 L CNN
+F 0 "C3" H 4050 2750 50  0000 L CNN
 F 1 "CP_Small" H 4050 2650 50  0000 L CNN
 F 2 "Capacitor_SMD:CP_Elec_5x4.4" H 4000 2700 50  0001 C CNN
@@
 	4350 3250 4350 3150
 $Comp
-L power:+5V #PWR?
+L power:+5V #PWR0105
 U 1 1 5BD034C4
 P 5600 2100
-F 0 "#PWR?" H 5600 1950 50  0001 C CNN
+F 0 "#PWR0105" H 5600 1950 50  0001 C CNN
 F 1 "+5V" H 5615 2273 50  0000 C CNN
 F 2 "" H 5600 2100 50  0001 C CNN
@@
 $EndComp
 $Comp
-L Device:R R?
+L Device:R R3
 U 1 1 5BD034CA
 P 5400 2300
-F 0 "R?" V 5500 2250 50  0000 C CNN
+F 0 "R3" V 5500 2250 50  0000 C CNN
 F 1 "10K" V 5500 2350 50  0000 C CNN
 F 2 "Resistor_SMD:R_0805_2012Metric" V 5330 2300 50  0001 C CNN
@@
 	5150 2300 5050 2300
 $Comp
-L power:GND #PWR?
+L power:GND #PWR0106
 U 1 1 5BD034DB
 P 4450 2400
-F 0 "#PWR?" H 4450 2150 50  0001 C CNN
+F 0 "#PWR0106" H 4450 2150 50  0001 C CNN
 F 1 "GND" H 4455 2227 50  0000 C CNN
 F 2 "" H 4450 2400 50  0001 C CNN
@@
 	4450 2300 4450 2400
 $Comp
-L Device:R_Small R?
+L Device:R_Small R5
 U 1 1 5BD034E6
 P 6450 4000
-F 0 "R?" V 6300 3900 50  0000 C CNN
+F 0 "R5" V 6300 3900 50  0000 C CNN
 F 1 "4K7" V 6350 4000 50  0000 C CNN
 F 2 "Resistor_SMD:R_0805_2012Metric" H 6450 4000 50  0001 C CNN
@@
 $EndComp
 $Comp
-L Device:R_Small R?
+L Device:R_Small R6
 U 1 1 5BD034ED
 P 6450 4100
-F 0 "R?" V 6500 4000 50  0000 C CNN
+F 0 "R6" V 6500 4000 50  0000 C CNN
 F 1 "4K7" V 6550 4100 50  0000 C CNN
 F 2 "Resistors_SMD:R_0805" H 6450 4100 50  0001 C CNN
@@
 	6000 4000 6350 4000
 $Comp
-L power:+5V #PWR?
+L power:+5V #PWR0107
 U 1 1 5BD034F6
 P 6750 4050
-F 0 "#PWR?" H 6750 3900 50  0001 C CNN
+F 0 "#PWR0107" H 6750 3900 50  0001 C CNN
 F 1 "+5V" H 6765 4223 50  0000 C CNN
 F 2 "" H 6750 4050 50  0001 C CNN
@@
 SGN1
 $Comp
-L Device:R_Small R?
+L Device:R_Small R4
 U 1 1 5BD03503
 P 6400 2700
-F 0 "R?" H 6300 2700 50  0000 C CNN
+F 0 "R4" H 6300 2700 50  0000 C CNN
 F 1 "10K" H 6250 2800 50  0000 C CNN
 F 2 "Resistor_SMD:R_0805_2012Metric" H 6400 2700 50  0001 C CNN
@@
 	6000 3050 6300 3050
 $Comp
-L Device:D_Zener_Small D?
+L Device:D_Zener_Small D4
 U 1 1 5BD0350C
 P 6550 2700
-F 0 "D?" V 6504 2768 50  0000 L CNN
+F 0 "D4" V 6504 2768 50  0000 L CNN
 F 1 "5.1V" V 6595 2768 50  0000 L CNN
 F 2 "Diodes_SMD:D_SMA" V 6550 2700 50  0001 C CNN
@@
 $EndComp
 $Comp
-L power:GND #PWR?
+L power:GND #PWR0108
 U 1 1 5BD03513
 P 6500 2850
-F 0 "#PWR?" H 6500 2600 50  0001 C CNN
+F 0 "#PWR0108" H 6500 2600 50  0001 C CNN
 F 1 "GND" H 6505 2677 50  0000 C CNN
 F 2 "" H 6500 2850 50  0001 C CNN
@@
 SGN2
 $Comp
-L Device:R_Small R?
+L Device:R_Small R8
 U 1 1 5BD03536
 P 6850 2950
-F 0 "R?" H 6750 2950 50  0000 C CNN
+F 0 "R8" H 6750 2950 50  0000 C CNN
 F 1 "1K" H 6700 3050 50  0000 C CNN
 F 2 "Resistor_SMD:R_0805_2012Metric" H 6850 2950 50  0001 C CNN
@@
 $EndComp
 $Comp
-L Device:D_Zener_Small D?
+L Device:D_Zener_Small D5
 U 1 1 5BD0353D
 P 7000 2950
-F 0 "D?" V 6954 3018 50  0000 L CNN
+F 0 "D5" V 6954 3018 50  0000 L CNN
 F 1 "5.1V" V 7045 3018 50  0000 L CNN
 F 2 "Diodes_SMD:D_SMA" V 7000 2950 50  0001 C CNN
@@
 $EndComp
 $Comp
-L power:GND #PWR?
+L power:GND #PWR0109
 U 1 1 5BD03544
 P 6950 3100
-F 0 "#PWR?" H 6950 2850 50  0001 C CNN
+F 0 "#PWR0109" H 6950 2850 50  0001 C CNN
 F 1 "GND" H 6955 2927 50  0000 C CNN
 F 2 "" H 6950 3100 50  0001 C CNN
@@
 	6650 2850 6850 2850
 $Comp
-L power:+5V #PWR?
+L power:+5V #PWR0110
 U 1 1 5BD03562
 P 7650 3450
-F 0 "#PWR?" H 7650 3300 50  0001 C CNN
+F 0 "#PWR0110" H 7650 3300 50  0001 C CNN
 F 1 "+5V" H 7665 3623 50  0000 C CNN
 F 2 "" H 7650 3450 50  0001 C CNN
@@
 $EndComp
 $Comp
-L power:GND #PWR?
+L power:GND #PWR0111
 U 1 1 5BD0357D
 P 7650 5050
-F 0 "#PWR?" H 7650 4800 50  0001 C CNN
+F 0 "#PWR0111" H 7650 4800 50  0001 C CNN
 F 1 "GND" H 7655 4877 50  0000 C CNN
 F 2 "" H 7650 5050 50  0001 C CNN
@@
 	6100 2950 6000 2950
 $Comp
-L Switch:SW_DIP_x04 SW?
+L Switch:SW_DIP_x04 SW3
 U 1 1 5BD035A0
 P 7300 3700
-F 0 "SW?" H 7300 4167 50  0000 C CNN
+F 0 "SW3" H 7300 4167 50  0000 C CNN
 F 1 "SW_DIP_x04" H 7300 4076 50  0000 C CNN
 F 2 "Button_Switch_THT:SW_DIP_SPSTx04_Slide_9.78x12.34mm_W7.62mm_P2.54mm" H 7300 3700 50  0001 C CNN
@@
 $EndComp
 $Comp
-L Device:C_Small C?
+L Device:C_Small C4
 U 1 1 5BD035AD
 P 4800 2550
-F 0 "C?" H 4650 2600 50  0000 L CNN
+F 0 "C4" H 4650 2600 50  0000 L CNN
 F 1 "C_Small" H 4550 2500 50  0000 L CNN
 F 2 "Capacitor_SMD:C_0805_2012Metric" H 4800 2550 50  0001 C CNN
@@
 	4550 2300 4450 2300
 $Comp
-L Device:LED D?
+L Device:LED D1
 U 1 1 5BD035BC
 P 4350 4250
-F 0 "D?" H 4342 3995 50  0000 C CNN
+F 0 "D1" H 4342 3995 50  0000 C CNN
 F 1 "LED" H 4342 4086 50  0000 C CNN
 F 2 "LED_SMD:LED_0805_2012Metric" H 4350 4250 50  0001 C CNN
@@
 $EndComp
 $Comp
-L Device:R_Small R?
+L Device:R_Small R1
 U 1 1 5BD035C3
 P 4000 4250
-F 0 "R?" H 3900 4250 50  0000 C CNN
+F 0 "R1" H 3900 4250 50  0000 C CNN
 F 1 "540" H 3850 4350 50  0000 C CNN
 F 2 "Resistor_SMD:R_0805_2012Metric" H 4000 4250 50  0001 C CNN
@@
 $EndComp
 $Comp
-L power:GND #PWR?
+L power:GND #PWR0112
 U 1 1 5BD035CA
 P 3800 4650
-F 0 "#PWR?" H 3800 4400 50  0001 C CNN
+F 0 "#PWR0112" H 3800 4400 50  0001 C CNN
 F 1 "GND" H 3805 4477 50  0000 C CNN
 F 2 "" H 3800 4650 50  0001 C CNN
@@
 $EndComp
 $Comp
-L Device:LED D?
+L Device:LED D2
 U 1 1 5BD035D0
 P 4350 4550
-F 0 "D?" H 4342 4295 50  0000 C CNN
+F 0 "D2" H 4342 4295 50  0000 C CNN
 F 1 "LED" H 4342 4386 50  0000 C CNN
 F 2 "LED_SMD:LED_0805_2012Metric" H 4350 4550 50  0001 C CNN
@@
 $EndComp
 $Comp
-L Device:R_Small R?
+L Device:R_Small R2
 U 1 1 5BD035D7
 P 4000 4550
-F 0 "R?" H 3900 4550 50  0000 C CNN
+F 0 "R2" H 3900 4550 50  0000 C CNN
 F 1 "540" H 3850 4650 50  0000 C CNN
 F 2 "Resistor_SMD:R_0805_2012Metric" H 4000 4550 50  0001 C CNN
@@
 ~SD
 $Comp
-L Device:D_Zener_Small D?
+L Device:D_Zener_Small D3
 U 1 1 5BD03602
 P 6400 5050
-F 0 "D?" V 6354 5118 50  0000 L CNN
+F 0 "D3" V 6354 5118 50  0000 L CNN
 F 1 "5.1V" V 6445 5118 50  0000 L CNN
 F 2 "LED_SMD:LED_0805_2012Metric" V 6400 5050 50  0001 C CNN
@@
 $EndComp
 $Comp
-L power:GND #PWR?
+L power:GND #PWR0113
 U 1 1 5BD03609
 P 6400 5150
-F 0 "#PWR?" H 6400 4900 50  0001 C CNN
+F 0 "#PWR0113" H 6400 4900 50  0001 C CNN
 F 1 "GND" H 6405 4977 50  0000 C CNN
 F 2 "" H 6400 5150 50  0001 C CNN
@@
 	6100 3350 6000 3350
 $Comp
-L Device:R_Small R?
+L Device:R_Small R7
 U 1 1 5BD252CE
 P 6750 2550
-F 0 "R?" H 6650 2550 50  0000 C CNN
+F 0 "R7" H 6650 2550 50  0000 C CNN
 F 1 "1K" H 6600 2650 50  0000 C CNN
 F 2 "Resistor_SMD:R_0805_2012Metric" H 6750 2550 50  0001 C CNN
@@
 	7150 2350 7300 2350
 $Comp
-L Switch:SW_Push SW?
+L Switch:SW_Push SW4
 U 1 1 5BD2C10B
 P 7450 5050
-F 0 "SW?" H 7450 5335 50  0000 C CNN
+F 0 "SW4" H 7450 5335 50  0000 C CNN
 F 1 "SW_Push" H 7450 5244 50  0000 C CNN
 F 2 "Button_Switch_THT:SW_PUSH_6mm" H 7450 5250 50  0001 C CNN
@@
 $EndComp
 $Comp
-L Switch:SW_Push SW?
+L Switch:SW_Push SW2
 U 1 1 5BD37D47
 P 6900 4550
-F 0 "SW?" H 6900 4835 50  0000 C CNN
+F 0 "SW2" H 6900 4835 50  0000 C CNN
 F 1 "SW_Push" H 6900 4744 50  0000 C CNN
 F 2 "Button_Switch_THT:SW_PUSH_6mm" H 6900 4750 50  0001 C CNN
@@
 $EndComp
 $Comp
-L power:GND #PWR?
+L power:GND #PWR0114
 U 1 1 5BD37DDD
 P 7100 4550
-F 0 "#PWR?" H 7100 4300 50  0001 C CNN
+F 0 "#PWR0114" H 7100 4300 50  0001 C CNN
 F 1 "GND" H 7105 4377 50  0000 C CNN
 F 2 "" H 7100 4550 50  0001 C CNN
@@
 $EndComp
 $Comp
-L Switch:SW_Push SW?
+L Switch:SW_Push SW1
 U 1 1 5BD38317
 P 4800 2300
-F 0 "SW?" H 4800 2585 50  0000 C CNN
+F 0 "SW1" H 4800 2585 50  0000 C CNN
 F 1 "SW_Push" H 4800 2494 50  0000 C CNN
 F 2 "Button_Switch_THT:SW_PUSH_6mm" H 4800 2500 50  0001 C CNN

Commit message: Sorted PCB
Parts:
- added R16: 4K7, Resistor_SMD:R_0805_2012Metric, symbol Device:R_Small
- added R20: 1K, Resistor_SMD:R_0805_2012Metric, symbol Device:R_Small
- R8: value 1K -> 10K
Connections:
- net +5V: now also R3.1, U1.4 (VCC), U1.6 (VCC); no longer R3.2
- net RST: now also R3.2; no longer R3.1
- net SCL: now also R5.2; no longer R6.2
- net SDA: now also R6.2; no longer R5.2
- net SGN2: now also R20.1; no longer D5.1 (K), R8.2, U1.14 ([10](OC1B/SS!)PB2)
- net ~SD: now also R16.1; no longer D3.1 (K), U1.11 ([7](AIN1)PD7)
- net Isense: now reaches U1.22 (A7)
- new net: D3.1 (K), R16.2, U1.11 ([7](AIN1)PD7)
- new net: D5.1 (K), R20.2, R8.2, U1.14 ([10](OC1B/SS!)PB2)
- no-connect marks 4 -> 3
Other:
- note removed: "I2C\n"
- note removed: "ISP"
- moved on the sheet: C1, C2, C3, C4, D4, D5, R3, R4, R5, R6, R7, R8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
