File: MosfetDriverOn2104/MosfetDriverOn210404.kicad_pcb (KiCad board)
At the start: 2 copper layers, 99.8 x 100.6 mm, 75 parts, among them J1 Screw_Terminal_01x02, J10 CROSS CONN, J11 servo hdr, J12 motor, J2 AVR-ISP-6, J3 I2C HDR, J4 I2C HDR, J5 UART HDR, J6 I2C HDR, J7 5V HDR, J8 ENCODER HDR, J9 GND HDR, Q1 IRF540N, Q2 IRF540N, Q3 IRF540N, Q4 IRF540N, SW1 SW_Push_Dual, SW2 SW1, SW3 SW2, SW4 SW_DIP_x04, U1 IR2104, U2 LM2576HVS-ADJ, U3 ATmega328P-AU-MCU_Microchip_A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, U4 L7805, U5 IR2104

Commit message: started routing
Parts:
- removed D14: D, Diode_SMD:D_SMA
- removed R20, R21, R22: R, Resistor_SMD:R_0805_2012Metric
- added C13: 22u, Capacitor_SMD:C_0805_2012Metric, F.Cu at (143.6, -3.86)
- added D8: D, Diode_SMD:D_SMA, F.Cu at (140.8, -6.61)
- added R12: R, Resistor_SMD:R_0805_2012Metric, F.Cu at (147.0, -5.12)
- added R14: R, Resistor_SMD:R_0805_2012Metric, F.Cu at (147.0, -3.17)
- added R15: R, Resistor_SMD:R_1206_3216Metric, F.Cu at (139.6, -3.69)
- added R16: R, Resistor_SMD:R_1206_3216Metric, F.Cu at (146.6, -7.24)
- C10, C9: value 22u -> CP; footprint Capacitor_SMD:C_0805_2012Metric -> Capacitor_SMD:CP_Elec_5x5.4
- C11: value 220uF -> C; footprint Capacitor_SMD:CP_Elec_5x4.4 -> Capacitor_SMD:C_0805_2012Metric
- C12: value 440uF -> 22u; footprint Capacitor_SMD:CP_Elec_5x4.4 -> Capacitor_SMD:C_0805_2012Metric
- C4: value CP -> C_Small; footprint Capacitor_SMD:CP_Elec_6.3x5.7 -> Capacitor_SMD:C_0805_2012Metric
- C5, C6: value CP -> 470; footprint Capacitor_SMD:CP_Elec_5x5.4 -> Capacitor_SMD:CP_Elec_8x6.2
- C7: value C -> CP; footprint Capacitor_SMD:C_0805_2012Metric -> Capacitor_SMD:CP_Elec_6.3x5.7
- C8: value .1uF -> CP; footprint Capacitor_SMD:C_0805_2012Metric -> Capacitor_SMD:CP_Elec_6.3x5.7
- CB2: value .1u -> 1uF
- CB3, CB5: value 1uF -> .1uF
- CB4: value .1uF -> 1uF
- CB6: value .1uF -> .1u
- D1, D2: value D -> LED; footprint Diode_SMD:D_SMA -> LED_SMD:LED_0805_2012Metric
- D10, D11: value 5.1V -> D; footprint Diodes_SMD:D_SMA -> Diode_SMD:D_SMA
- D3: value D -> 5.1V; footprint Diode_SMD:D_SMA -> LED_SMD:LED_0805_2012Metric
- D4: value SS24 -> 5.1V
- D5: value LED -> 5.1V
- D6: value LED -> SS24; footprint LED_SMD:LED_0805_2012Metric -> Diode_SMD:D_SMA
- D7: value 5.1V -> POWER_LED; footprint Diode_SMD:D_SMA -> LED_SMD:LED_0805_2012Metric
- D9: value POWER_LED -> D; footprint LED_SMD:LED_0805_2012Metric -> Diode_SMD:D_SMA
- J1: value Screw_Terminal_01x02 -> I2C HDR; footprint TerminalBlock:TerminalBlock_Altech_AK300-2_P5.00mm -> Connector_PinHeader_2.54mm:PinHeader_1x04_P2.54mm_Vertical
- J10: value CROSS CONN -> ENCODER HDR
- J11: value servo hdr -> CROSS CONN; footprint TerminalBlock:TerminalBlock_Altech_AK300-3_P5.00mm -> Connector_PinHeader_2.54mm:PinHeader_2x02_P2.54mm_Vertical
- J2: footprint Connector_PinHeader_2.54mm:PinHeader_2x03_P2.54mm_Vertical -> Connector_PinHeader_2.54mm:PinHeader_1x04_P2.54mm_Vertical
- J4: value I2C HDR -> Screw_Terminal_01x02; footprint Connector_PinHeader_2.54mm:PinHeader_1x04_P2.54mm_Vertical -> TerminalBlock:TerminalBlock_Altech_AK300-2_P5.00mm
- J5: value UART HDR -> I2C HDR
- J6: value I2C HDR -> UART HDR
- J8: value ENCODER HDR -> GND HDR
- J9: value GND HDR -> servo hdr; footprint Connector_PinHeader_2.54mm:PinHeader_1x04_P2.54mm_Vertical -> TerminalBlock:TerminalBlock_Altech_AK300-3_P5.00mm
- R1, R2: value R -> 540
- R10: value 540 -> 2k7
- R13: value 1K -> R
- R18, R19: footprint Resistor_SMD:R_1206_3216Metric -> Resistor_SMD:R_0805_2012Metric
- R3: value 240 -> 10K
- R4: value 2k7 -> 10K
- R5: value 10K -> 4K7
- R6: value 1K -> 4K7
- R7: value 4K7 -> 1K
- R8: value 4K7 -> 1K; footprint Resistors_SMD:R_0805 -> Resistor_SMD:R_0805_2012Metric
- R9: value 540 -> 240
- SW1: value SW_Push_Dual -> SW_Push; footprint Button_Switch_THT:SW_TH_Tactile_Omron_B3F-10xx -> Button_Switch_THT:SW_PUSH_6mm
- SW2: value SW1 -> SW_Push; footprint Button_Switch_THT:SW_TH_Tactile_Omron_B3F-10xx -> Button_Switch_THT:SW_PUSH_6mm
- SW3: value SW2 -> SW_DIP_x04; footprint Button_Switch_THT:SW_TH_Tactile_Omron_B3F-10xx -> Button_Switch_THT:SW_DIP_SPSTx04_Slide_9.78x12.34mm_W7.62mm_P2.54mm
- SW4: value SW_DIP_x04 -> SW_Push; footprint Button_Switch_THT:SW_DIP_SPSTx04_Slide_9.78x12.34mm_W7.62mm_P2.54mm -> Button_Switch_THT:SW_PUSH_6mm
- U1: value IR2104 -> ATmega328P-AU-MCU_Microchip_ATmega; footprint Package_DIP:DIP-8_W7.62mm_Socket_LongPads -> Package_QFP:TQFP-32_7x7mm_P0.8mm
- U3: value ATmega328P-AU-MCU_Microchip_ATmega -> L7805; footprint Package_QFP:TQFP-32_7x7mm_P0.8mm -> Package_TO_SOT_SMD:TO-263-2
- U4: value L7805 -> IR2104; footprint Package_TO_SOT_SMD:TO-263-3_TabPin2 -> Package_DIP:DIP-8_W7.62mm_Socket_LongPads
- moved R7 89.5 mm to (129.4, -119.3), turned to 270 degrees
- moved R5 89.2 mm to (158.6, -124.8)
- moved CB4 82.5 mm to (83.7, -52.9), turned to 270 degrees
- moved R1 82.1 mm to (92.8, -14.4), turned to 90 degrees
- moved C9 81.1 mm to (81.7, -52.9), turned to 270 degrees
- moved D1 74.7 mm to (74.8, -59.4), turned to 180 degrees
- moved D2 74.4 mm to (89.8, -15.1), turned to 270 degrees
- moved R11 71.9 mm to (206.7, -66.3)
- moved R10 68.1 mm to (93.6, -67.3)
- moved U3 64.2 mm to (127.1, -109.5)
- moved R2 62.0 mm to (108.5, -16.8)
- moved R13 60.8 mm to (201.5, -49.1)
- moved R8 57.5 mm to (127.4, -119.3), turned to 270 degrees
- moved D10 55.5 mm to (164.8, -45.0), turned to 180 degrees
- moved D12 55.4 mm to (71.7, -25.0)
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Connections:
- net /M1 renamed /H-bridge/M1
- net /M2 renamed /H-bridge/M2
- C10 pad 1: Net-(C10-Pad1) -> +5V
- C10 pad 2: Net-(C10-Pad2) -> GND
- C11 pad 1: VCC -> +5V
- C12 pad 1: VCC -> Net-(C12-Pad1)
- C12 pad 2: GND -> Net-(C12-Pad2)
- C4 pad 1: +15V -> /controller/RST
- C5 pad 1: +15V -> VCC
- C6 pad 1: +5V -> VCC
- C7 pad 1: +5V -> VCC
- C8 pad 1: /RST -> +15V
- C9 pad 1: Net-(C9-Pad1) -> +15V
- C9 pad 2: Net-(C9-Pad2) -> GND
- CB1 pad 1: Net-(C9-Pad1) -> Net-(C12-Pad1)
- CB1 pad 2: Net-(C9-Pad2) -> Net-(C12-Pad2)
- CB2 pad 1: Net-(C10-Pad1) -> +15V
- CB2 pad 2: Net-(C10-Pad2) -> GND
- CB6 pad 1: +15V -> Net-(C13-Pad1)
- CB6 pad 2: GND -> Net-(C13-Pad2)
- D1 pad 1: Net-(C9-Pad1) -> Net-(D1-Pad1)
- D1 pad 2: +15V -> Net-(D1-Pad2)
- D10 pad 1: /SGN1 -> Net-(D10-Pad1)
- D10 pad 2: GND -> Net-(D10-Pad2)
- D11 pad 1: /SGN2 -> Net-(D11-Pad1)
- D11 pad 2: GND -> Net-(D11-Pad2)
- D13 pad 1: Net-(D13-Pad1) -> Net-(C13-Pad1)
- D13 pad 2: Net-(D13-Pad2) -> +15V
- D3 pad 1: Net-(D3-Pad1) -> /controller/~SD
- D3 pad 2: Net-(D3-Pad2) -> GND
- D5 pad 1: Net-(D5-Pad1) -> /controller/SGN2
- D5 pad 2: Net-(D5-Pad2) -> GND
- D6 pad 2: Net-(D6-Pad2) -> GND
- D7 pad 1: /~SD -> Net-(D7-Pad1)
- D7 pad 2: GND -> +5V
- D9 pad 2: +5V -> Net-(D9-Pad2)
- J1 pad 2: VCC -> /Sheet5BD0E603/SCL
- J10 pad 1: /SGN1 -> GND
- J10 pad 2: /IN1 -> (no net)
- J10 pad 3: /IN2 -> (no net)
- J10 pad 4: /SGN2 -> +5V
- J11 pad 1: GND -> (no net)
- J11 pad 2: /svo -> /H-bridge/IN1
- J11 pad 3: +5V -> /H-bridge/IN2
- J2 pad 1: /MISO -> (no net)
- J2 pad 3: /SCK -> (no net)
- J2 pad 4: /MOSI -> (no net)
- J3 pad 2: /SCL -> /Sheet5BD0E603/SCL
- J3 pad 3: /SDA -> /Sheet5BD0E603/SDA
- J4 pad 2: /SCL -> VCC
- J5 pad 2: /TX -> /Sheet5BD0E603/SCL
- J5 pad 3: /RX -> /Sheet5BD0E603/SDA
- J6 pad 2: /SCL -> (no net)
- J6 pad 3: /SDA -> (no net)
- J8 pad 2: /B -> GND
- J8 pad 3: /A -> GND
- J8 pad 4: +5V -> GND
- J9 pad 2: GND -> (no net)
- J9 pad 3: GND -> +5V
- L1 pad 1: Net-(D4-Pad1) -> Net-(D6-Pad1)
- Q1 pad 1: Net-(D2-Pad2) -> Net-(D9-Pad2)
- Q2 pad 1: Net-(D3-Pad2) -> Net-(D10-Pad2)
- Q2 pad 3: /IS+ -> /H-bridge/IS+
- Q3 pad 1: Net-(D12-Pad2) -> Net-(D11-Pad2)
- Q4 pad 1: Net-(D13-Pad2) -> Net-(D12-Pad2)
- Q4 pad 3: /IS+ -> /H-bridge/IS+
- R1 pad 1: Net-(D2-Pad2) -> Net-(D1-Pad1)
- R1 pad 2: Net-(D2-Pad1) -> GND
- R10 pad 1: Net-(D5-Pad1) -> Net-(R10-Pad1)
- R11 pad 1: Net-(D6-Pad1) -> GND
- R11 pad 2: GND -> Net-(D7-Pad1)
- R13 pad 1: GND -> Net-(D9-Pad2)
- R13 pad 2: /SGN2 -> Net-(D9-Pad1)
- R17 pad 1: /~SD -> Net-(D11-Pad2)
- R17 pad 2: +5V -> Net-(D11-Pad1)
- R18 pad 1: /IS+ -> Net-(D12-Pad2)
- R18 pad 2: GND -> Net-(D12-Pad1)
- R19 pad 1: /IS+ -> /H-bridge/~SD
- R19 pad 2: GND -> +5V
- R2 pad 1: Net-(D3-Pad2) -> Net-(D2-Pad1)
- R2 pad 2: Net-(D3-Pad1) -> GND
- R3 pad 1: Net-(R3-Pad1) -> /controller/RST
- R3 pad 2: +15V -> +5V
- R4 pad 1: Net-(R3-Pad1) -> GND
- R4 pad 2: GND -> Net-(D4-Pad1)
- R5 pad 1: /RST -> +5V
- R5 pad 2: +5V -> /controller/SDA
- R6 pad 1: GND -> +5V
- R6 pad 2: /SGN1 -> /controller/SCL
- R7 pad 1: +5V -> (no net)
- R7 pad 2: /SDA -> Net-(D4-Pad1)
- R8 pad 1: +5V -> GND
- R8 pad 2: /SCL -> /controller/SGN2
- R9 pad 1: GND -> Net-(R10-Pad1)
- R9 pad 2: Net-(D9-Pad1) -> +15V
- SW1 pad 2: /RST -> /controller/RST
- SW2 pad 1: +5V -> Net-(SW2-Pad1)
- SW3 pad 1: +5V -> Net-(SW3-Pad1)
- SW3 pad 2: GND -> Net-(SW3-Pad2)
- SW3 pad 3: +5V -> Net-(SW3-Pad3)
- SW3 pad 4: GND -> Net-(SW3-Pad4)
- SW4 pad 2: Net-(SW4-Pad2) -> GND
- U1 pad 1: +15V -> (no net)
- U1 pad 2: /IN1 -> Net-(SW2-Pad1)
- U1 pad 3: /~SD -> GND
- U1 pad 4: GND -> +5V
- U1 pad 5: Net-(D3-Pad1) -> GND
- U1 pad 6: Net-(C9-Pad2) -> +5V
- U1 pad 7: Net-(D2-Pad1) -> Net-(D1-Pad2)
- U1 pad 8: Net-(C9-Pad1) -> Net-(D2-Pad2)
- U2 pad 2: Net-(D4-Pad1) -> Net-(D6-Pad1)
- U2 pad 4: Net-(R3-Pad1) -> Net-(R10-Pad1)
- U3 pad 1: /B -> +15V
- U3 pad 2: +5V -> GND
- U3 pad 3: GND -> +5V
- U4 pad 2: GND -> /H-bridge/IN1
- U4 pad 3: +5V -> /H-bridge/~SD
- U5 pad 2: /IN2 -> /H-bridge/IN2
- U5 pad 3: /~SD -> /H-bridge/~SD
- U5 pad 5: Net-(D13-Pad1) -> Net-(D12-Pad1)
- U5 pad 6: Net-(C10-Pad2) -> Net-(C13-Pad2)
- U5 pad 7: Net-(D12-Pad1) -> Net-(D11-Pad1)
- U5 pad 8: Net-(C10-Pad1) -> Net-(C13-Pad1)

Commit message: Sorted PCB
Parts:
- removed R16: R, Resistor_SMD:R_1206_3216Metric
- added C14: C_Small, Capacitor_SMD:C_0805_2012Metric, F.Cu at (187.7, 9.65)
- added C15: C_Small, Capacitor_SMD:C_0805_2012Metric, F.Cu at (179.8, 9.78)
- added C16: 470, Capacitor_SMD:CP_Elec_8x6.2, F.Cu at (41.8, -54.7)
- added C17: 470, Capacitor_SMD:CP_Elec_10x7.9, F.Cu at (-1.51, -14.4)
- added C18: 470, Capacitor_SMD:CP_Elec_10x7.9, F.Cu at (12.1, -14.4)
- added R20: 4K7, Resistor_SMD:R_0805_2012Metric, F.Cu at (181.9, -20.0)
- added R21: 4K7, Resistor_SMD:R_0805_2012Metric, F.Cu at (183.2, -21.4)
- added R22: 4K7, Resistor_SMD:R_0805_2012Metric, F.Cu at (196.2, 1.04)
- added R23: 10K, Resistor_SMD:R_0805_2012Metric, F.Cu at (204.2, -2.03)
- added R24: 10K, Resistor_SMD:R_0805_2012Metric, F.Cu at (212.9, -2.01)
- added R25: 1K, Resistor_SMD:R_0805_2012Metric, F.Cu at (204.2, -5.51)
- added R26: 1K, Resistor_SMD:R_0805_2012Metric, F.Cu at (212.9, -5.46)
- added U6: ATmega328P-AU-MCU_Microchip_ATmega, Package_QFP:TQFP-32_7x7mm_P0.8mm, F.Cu at (188.3, -12.8)
- C1, C2: value C_Small -> 470; footprint Capacitor_SMD:C_0805_2012Metric -> Capacitor_SMD:CP_Elec_8x6.2
- C10: value CP -> C_Small; footprint Capacitor_SMD:CP_Elec_5x5.4 -> Capacitor_SMD:C_0805_2012Metric
- C11: value C -> CP_Small; footprint Capacitor_SMD:C_0805_2012Metric -> Capacitor_SMD:CP_Elec_5x4.4
- C12, C13: value 22u -> C_Small
- C3: value CP_Small -> CP; footprint Capacitor_SMD:CP_Elec_5x4.4 -> Capacitor_SMD:CP_Elec_6.3x5.7
- C4: value C_Small -> CP; footprint Capacitor_SMD:C_0805_2012Metric -> Capacitor_SMD:CP_Elec_6.3x5.7
- C5, C6: value 470 -> CP; footprint Capacitor_SMD:CP_Elec_8x6.2 -> Capacitor_SMD:CP_Elec_5x5.4
- C7: value CP -> C; footprint Capacitor_SMD:CP_Elec_6.3x5.7 -> Capacitor_SMD:C_0805_2012Metric
- C8: value CP -> 22u; footprint Capacitor_SMD:CP_Elec_6.3x5.7 -> Capacitor_SMD:CP_Elec_4x4.5
- C9: value CP -> 22u; footprint Capacitor_SMD:CP_Elec_5x5.4 -> Capacitor_SMD:CP_Elec_4x4.5
- D1: value LED -> SS24; footprint LED_SMD:LED_0805_2012Metric -> Diode_SMD:D_SMC
- D10, D9: value D -> LED; footprint Diode_SMD:D_SMA -> LED_SMD:LED_0805_2012Metric
- D11, D12, D13: value D -> 5.1V; footprint Diode_SMD:D_SMA -> Diode_THT:D_A-405_P7.62mm_Horizontal
- D2: value LED -> POWER_LED
- D3, D5: value 5.1V -> D; footprint LED_SMD:LED_0805_2012Metric -> Diode_SMD:D_SMA
- D4: value 5.1V -> D
- D6: value SS24 -> D
- D7: value POWER_LED -> D; footprint LED_SMD:LED_0805_2012Metric -> Diode_SMD:D_SMA
- J2: footprint Connector_PinHeader_2.54mm:PinHeader_1x04_P2.54mm_Vertical -> Connector_PinHeader_2.54mm:PinHeader_2x03_P2.54mm_Vertical
- J9: footprint TerminalBlock:TerminalBlock_Altech_AK300-3_P5.00mm -> Connector_PinSocket_2.54mm:PinSocket_1x03_P2.54mm_Vertical
- R1: value 540 -> 240
- R10: value 2k7 -> 1K
- R11: value 540 -> 0E05; footprint Resistor_SMD:R_0805_2012Metric -> Resistor_SMD:R_1206_3216Metric
- R12: value R -> 0E05; footprint Resistor_SMD:R_0805_2012Metric -> Resistor_SMD:R_1206_3216Metric
- R13, R19: value R -> 10K
- R15: footprint Resistor_SMD:R_1206_3216Metric -> Resistor_SMD:R_0805_2012Metric
- R17, R18: value R -> 540
- R2: value 540 -> 2k7
- R3: value 10K -> 540
- R4: value 10K -> R
- R5, R6: value 4K7 -> R
- R7, R8: value 1K -> 0E05; footprint Resistor_SMD:R_0805_2012Metric -> Resistor_SMD:R_1206_3216Metric
- R9: value 240 -> 0E05; footprint Resistor_SMD:R_0805_2012Metric -> Resistor_SMD:R_1206_3216Metric
- SW2: value SW_Push -> SW_DIP_x04; footprint Button_Switch_THT:SW_PUSH_6mm -> Button_Switch_THT:SW_DIP_SPSTx04_Slide_9.78x12.34mm_W7.62mm_P2.54mm
- SW3: value SW_DIP_x04 -> SW_Push; footprint Button_Switch_THT:SW_DIP_SPSTx04_Slide_9.78x12.34mm_W7.62mm_P2.54mm -> Button_Switch_THT:SW_PUSH_6mm
- U1: value ATmega328P-AU-MCU_Microchip_ATmega -> LM2576HVS-ADJ; footprint Package_QFP:TQFP-32_7x7mm_P0.8mm -> Package_TO_SOT_SMD:TO-263-5_TabPin3
- U2: value LM2576HVS-ADJ -> L7805; footprint Package_TO_SOT_SMD:TO-263-5_TabPin3 -> Package_TO_SOT_SMD:TO-263-2
- U3: value L7805 -> IR2104; footprint Package_TO_SOT_SMD:TO-263-2 -> Package_DIP:DIP-8_W7.62mm_Socket_LongPads
- U4: value IR2104 -> LM358; footprint Package_DIP:DIP-8_W7.62mm_Socket_LongPads -> Package_SO:SOIC-8_3.9x4.9mm_P1.27mm
- moved C5 193.7 mm to (37.0, -63.1)
- moved R4 188.7 mm to (196.2, 4.55), turned to 270 degrees
- moved C3 185.1 mm to (-23.1, -23.6)
- moved J7 176.1 mm to (80.8, 96.3), turned to 90 degrees
- moved CB1 167.9 mm to (37.5, 16.5), turned to 270 degrees
- moved J8 161.8 mm to (88.5, 88.3), turned to 90 degrees
- moved C6 160.6 mm to (79.7, 85.7)
- moved U3 159.9 mm to (34.6, 20.9)
- moved C8 159.6 mm to (42.5, 16.6), turned to 180 degrees
- moved J4 157.8 mm to (-25.3, -68.8), turned to 180 degrees
- moved CB3 157.0 mm to (32.5, -9.91)
- moved CB5 155.6 mm to (20.0, -46.5), turned to 180 degrees
- moved CB4 149.6 mm to (54.3, 93.8), turned to 90 degrees
- moved CB6 147.0 mm to (39.0, -15.6), turned to 180 degrees
- moved R9 138.4 mm to (113.5, -32.6)
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Connections:
- net /H-bridge/IN2 renamed /IN2
- net /H-bridge/M1 renamed /M1
- net /H-bridge/M2 renamed /M2
- net /Sheet5BD0E603/SCL renamed /SCL
- net /Sheet5BD0E603/SDA renamed /SDA
- C1 pad 1: +5V -> VCC
- C10 pad 1: +5V -> /RST
- C12 pad 1: Net-(C12-Pad1) -> +5V
- C12 pad 2: Net-(C12-Pad2) -> GND
- C13 pad 1: Net-(C13-Pad1) -> +5V
- C13 pad 2: Net-(C13-Pad2) -> GND
- C2 pad 1: +5V -> VCC
- C3 pad 1: +5V -> VCC
- C4 pad 1: /controller/RST -> +15V
- C5 pad 1: VCC -> +15V
- C6 pad 1: VCC -> +5V
- C7 pad 1: VCC -> +5V
- C8 pad 1: +15V -> Net-(C8-Pad1)
- C8 pad 2: GND -> Net-(C8-Pad2)
- C9 pad 1: +15V -> Net-(C9-Pad1)
- C9 pad 2: GND -> Net-(C9-Pad2)
- CB1 pad 1: Net-(C12-Pad1) -> Net-(C8-Pad1)
- CB1 pad 2: Net-(C12-Pad2) -> Net-(C8-Pad2)
- CB6 pad 1: Net-(C13-Pad1) -> Net-(C9-Pad1)
- CB6 pad 2: Net-(C13-Pad2) -> Net-(C9-Pad2)
- D1 pad 2: Net-(D1-Pad2) -> GND
- D11 pad 2: Net-(D11-Pad2) -> GND
- D12 pad 2: Net-(D12-Pad2) -> GND
- D13 pad 1: Net-(C13-Pad1) -> Net-(D13-Pad1)
- D13 pad 2: +15V -> GND
- D2 pad 2: Net-(D2-Pad2) -> +5V
- D3 pad 1: /controller/~SD -> Net-(C8-Pad1)
- D3 pad 2: GND -> +15V
- D4 pad 2: GND -> Net-(D4-Pad2)
- D5 pad 1: /controller/SGN2 -> Net-(D5-Pad1)
- D5 pad 2: GND -> Net-(D5-Pad2)
- D6 pad 2: GND -> Net-(D6-Pad2)
- D7 pad 2: +5V -> Net-(D7-Pad2)
- D8 pad 1: Net-(C12-Pad1) -> Net-(C9-Pad1)
- J10 pad 2: (no net) -> /B
- J10 pad 3: (no net) -> /A
- J11 pad 1: (no net) -> /SGN1
- J11 pad 2: /H-bridge/IN1 -> /IN1
- J11 pad 4: (no net) -> /SGN2
- J2 pad 1: (no net) -> /MISO
- J2 pad 3: (no net) -> /SCK
- J2 pad 4: (no net) -> /MOSI
- J6 pad 2: (no net) -> /TX
- J6 pad 3: (no net) -> /RX
- J9 pad 2: (no net) -> +5V
- J9 pad 3: +5V -> /svo
- L1 pad 1: Net-(D6-Pad1) -> Net-(D1-Pad1)
- Q1 pad 1: Net-(D9-Pad2) -> Net-(D4-Pad2)
- Q2 pad 1: Net-(D10-Pad2) -> Net-(D5-Pad2)
- Q2 pad 3: /H-bridge/IS+ -> /IS+
- Q3 pad 1: Net-(D11-Pad2) -> Net-(D6-Pad2)
- Q4 pad 1: Net-(D12-Pad2) -> Net-(D7-Pad2)
- Q4 pad 3: /H-bridge/IS+ -> /IS+
- R1 pad 1: Net-(D1-Pad1) -> Net-(R1-Pad1)
- R1 pad 2: GND -> +15V
- R11 pad 1: GND -> /IS+
- R11 pad 2: Net-(D7-Pad1) -> GND
- R12 pad 1: /H-bridge/~SD -> /IS+
- R12 pad 2: +5V -> GND
- R13 pad 1: Net-(D9-Pad2) -> Net-(R10-Pad1)
- R13 pad 2: Net-(D9-Pad1) -> /Isense
- R14 pad 1: Net-(D10-Pad2) -> Net-(D6-Pad2)
- R14 pad 2: Net-(D10-Pad1) -> Net-(D6-Pad1)
- R15 pad 1: /H-bridge/IS+ -> Net-(D7-Pad2)
- R15 pad 2: GND -> Net-(D7-Pad1)
- R17 pad 1: Net-(D11-Pad2) -> Net-(D9-Pad1)
- R17 pad 2: Net-(D11-Pad1) -> GND
- R18 pad 1: Net-(D12-Pad2) -> Net-(D10-Pad1)
- R18 pad 2: Net-(D12-Pad1) -> GND
- R19 pad 1: /H-bridge/~SD -> +5V
- R19 pad 2: +5V -> /RST
- R2 pad 1: Net-(D2-Pad1) -> Net-(R1-Pad1)
- R3 pad 1: /controller/RST -> GND
- R3 pad 2: +5V -> Net-(D2-Pad1)
- R4 pad 1: GND -> /~SD
- R4 pad 2: Net-(D4-Pad1) -> +5V
- R5 pad 1: +5V -> Net-(D4-Pad2)
- R5 pad 2: /controller/SDA -> Net-(D4-Pad1)
- R6 pad 1: +5V -> Net-(D5-Pad2)
- R6 pad 2: /controller/SCL -> Net-(D5-Pad1)
- R7 pad 1: (no net) -> /IS+
- R7 pad 2: Net-(D4-Pad1) -> GND
- R8 pad 1: GND -> /IS+
- R8 pad 2: /controller/SGN2 -> GND
- R9 pad 1: Net-(R10-Pad1) -> /IS+
- R9 pad 2: +15V -> GND
- SW1 pad 2: /controller/RST -> /RST
- SW2 pad 2: GND -> Net-(SW2-Pad2)
- SW3 pad 1: Net-(SW3-Pad1) -> Net-(C14-Pad1)
- SW3 pad 2: Net-(SW3-Pad2) -> GND
- SW4 pad 1: Net-(SW4-Pad1) -> Net-(C15-Pad1)
- U1 pad 1: (no net) -> VCC
- U1 pad 2: Net-(SW2-Pad1) -> Net-(D1-Pad1)
- U1 pad 4: +5V -> Net-(R1-Pad1)
- U2 pad 1: VCC -> +15V
- U2 pad 2: Net-(D6-Pad1) -> GND
- U2 pad 3: GND -> +5V
- U3 pad 2: GND -> /IN1
- U3 pad 3: +5V -> /~SD
- U4 pad 1: +15V -> /Isense
- U4 pad 2: /H-bridge/IN1 -> Net-(R10-Pad1)
- U4 pad 3: /H-bridge/~SD -> /IS+
- U4 pad 5: Net-(D10-Pad1) -> GND
- U4 pad 6: Net-(C12-Pad2) -> GND
- U4 pad 7: Net-(D9-Pad1) -> (no net)
- U4 pad 8: Net-(C12-Pad1) -> +5V
- U5 pad 3: /H-bridge/~SD -> /~SD
- U5 pad 5: Net-(D12-Pad1) -> Net-(D7-Pad1)
- U5 pad 6: Net-(C13-Pad2) -> Net-(C9-Pad2)
- U5 pad 7: Net-(D11-Pad1) -> Net-(D6-Pad1)
- U5 pad 8: Net-(C13-Pad1) -> Net-(C9-Pad1)

Commit message: Arrenged components,just need to pack a little bit tighter
Parts:
- removed C3: CP, Capacitor_SMD:CP_Elec_6.3x5.7
- C8, C9: footprint Capacitor_SMD:CP_Elec_4x4.5 -> Capacitor_SMD:CP_Elec_5x5.3
- moved C15 181.8 mm to (-2.01, 11.8)
- moved D11 181.8 mm to (11.5, 2.24)
- moved R21 181.8 mm to (1.42, -19.4)
- moved SW4 181.8 mm to (-4.09, 9.14)
- moved C10 181.8 mm to (24.4, -17.8)
- moved C13 181.8 mm to (20.5, -19.1)
- moved C14 181.8 mm to (5.87, 11.7)
- moved C7 181.8 mm to (0.86, -5.28)
- moved D10 181.8 mm to (5.06, 0.03)
- moved D12 181.8 mm to (25.0, -5.16)
- moved D13 181.8 mm to (28.4, -5.16)
- moved D9 181.8 mm to (5.09, -2.01)
- moved J1 181.8 mm to (-6.39, -26.7)
- moved J10 181.8 mm to (-10.5, -0.61)
- moved J2 181.8 mm to (16.0, -15.5)
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
Commit message: Started tightening board
Parts:
- moved C10 219.8 mm to (123.8, 178.2)
- moved C13 219.8 mm to (120.0, 176.9)
- moved C14 219.8 mm to (105.3, 207.7)
- moved C15 219.8 mm to (97.5, 207.8)
- moved C7 219.8 mm to (100.3, 190.7)
- moved D11 219.8 mm to (110.9, 198.2)
- moved D12 219.8 mm to (124.5, 190.8)
- moved D13 219.8 mm to (127.9, 190.8)
- moved D9 219.8 mm to (104.6, 194.0)
- moved J1 219.8 mm to (93.1, 169.3)
- moved J10 219.8 mm to (89.0, 195.4)
- moved J2 219.8 mm to (115.5, 180.5)
- moved J3 219.8 mm to (93.1, 162.0)
- moved J5 219.8 mm to (93.1, 165.6)
- moved J6 219.8 mm to (88.6, 180.9)
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